File: PCB_electronics/power_controller/power_controller.kicad_pcb (KiCad board)
At the start: 2 copper layers, 20 parts, among them IC1 ATMEGA328-P, P1 SOLAR_PANEL, P2 5V_pololu, P3 BATT, P4 SUPERCAPS, P5 PWR_MEGA, P6 FEEDBACK_MEGA, U1 IRLB-8721_SOL, U2 IRLB-8721_MEGA, Y1 16MHz

Commit message: first version of power controller
Parts:
- removed P1: SOLAR_PANEL, Wire_Connections_Bridges:WireConnection_2.00mmDrill
- removed P2: 5V_pololu, Wire_Connections_Bridges:WireConnection_2.00mmDrill
- removed P3: BATT, Wire_Connections_Bridges:WireConnection_2.00mmDrill
- removed P4: SUPERCAPS, Wire_Connections_Bridges:WireConnection_2.00mmDrill
- removed P5: PWR_MEGA, Wire_Connections_Bridges:WireConnection_2.00mmDrill
- removed P6: FEEDBACK_MEGA, Wire_Pads:SolderWirePad_single_1-2mmDrill
- added BATT: BATT, Wire_Connections_Bridges:WireConnection_2.00mmDrill, F.Cu at (105.0, 44.0)
- added CAPS: SUPERCAPS, Wire_Connections_Bridges:WireConnection_2.00mmDrill, F.Cu at (85.0, 90.0)
- added FBK: FEEDBACK_MEGA, Wire_Pads:SolderWirePad_single_1-2mmDrill, F.Cu at (84.0, 51.0)
- added MEGA: PWR_MEGA, Wire_Connections_Bridges:WireConnection_2.00mmDrill, F.Cu at (86.0, 44.0)
- added POLOLU: 5V_pololu, Wire_Connections_Bridges:WireConnection_2.00mmDrill, F.Cu at (85.0, 70.0)
- added SOL: SOLAR_PANEL, Wire_Connections_Bridges:WireConnection_2.00mmDrill, F.Cu at (125.0, 44.0)
- IC1: footprint Housings_DIP:DIP-28_W15.24mm_LongPads -> Housings_DIP:DIP-28_W7.62mm_LongPads
- R1, R2, R3, R4, R5, R6, R7: footprint Resistors_ThroughHole:Resistor_Horizontal_RM20mm -> Resistors_ThroughHole:Resistor_Horizontal_RM10mm
- moved R1 98.9 mm to (128.0, 91.0), turned to 90 degrees
- moved C2 59.8 mm to (97.5, 96.0), turned to 180 degrees
- moved Y1 59.4 mm to (97.0, 105.0)
- moved C1 58.4 mm to (96.0, 115.0)
- moved R3 55.0 mm to (95.0, 70.0)
- moved R6 53.2 mm to (104.0, 60.0), turned to 180 degrees
- moved R2 47.7 mm to (128.0, 76.0), turned to 90 degrees
- moved IC1 46.8 mm to (105.0, 78.0)
- moved U2 46.2 mm to (99.0, 53.0), turned to 180 degrees
- moved U1 46.0 mm to (115.0, 53.0), turned to 180 degrees
- moved R7 43.1 mm to (98.0, 88.0), turned to 90 degrees
- moved R4 43.0 mm to (118.0, 100.0)
- moved R5 41.6 mm to (120.0, 60.0), turned to 180 degrees
- moved D1 15.4 mm to (135.0, 97.0), turned to 270 degrees
Connections:
- IC1 pad 21: +5V -> Net-(IC1-Pad21)
Routing:
- net +5V: track 0.00 -> 136.1 mm
- net /D5: track 0.00 -> 129.2 mm
- net /A0: track 0.00 -> 72.9 mm
- net /D3: track 0.00 -> 71.1 mm, vias 0 -> 1
- net /MEGA_FBK: track 0.00 -> 65.9 mm
- net /MSFT_SOLAR_S: track 0.00 -> 58.1 mm
- net /A1: track 0.00 -> 23.3 mm
- net Net-(C1-Pad1): track 0.00 -> 18.8 mm
- net Net-(C2-Pad1): track 0.00 -> 14.5 mm
- net GND: track 0.00 -> 10.5 mm
- net /MEGA-: track 0.00 -> 9.12 mm
- net Net-(IC1-Pad1): track 0.00 -> 8.07 mm
- net Net-(D1-Pad2): track 0.00 -> 7.03 mm
- net Net-(IC1-Pad19): track 0.00 -> 5.74 mm
- added copper zone on B.Cu, net GND
Other:
- board outline added: 60 x 80 mm
- net class Default: clearance 0.2 -> 0.3
- net class power added: clearance 0.3, trace_width 0.75, via_dia 0.9, via_drill 0.6
- rule pad_to_mask_clearance: 0.2 -> 0
- rule trace_clearance: 0.2 -> 0.3
- board text added: "+"
- board text added: "-"

Commit message: some stupid changes
Parts:
- renumbered SOL to P1, POLOLU to P2, BATT to P3, CAPS to P4, MEGA to P5, FBK to P6
Changed lines of the file:
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@@
     (links 38)
     (no_connects 0)
-    (area 79.949999 39.949999 140.050001 120.050001)
+    (area 76 37 147.000001 123.000001)
     (thickness 1.6)
     (drawings 15)
@@
     (39 F.Mask user)
     (40 Dwgs.User user)
-    (41 Cmts.User user)
+    (41 Cmts.User user hide)
     (42 Eco1.User user)
     (43 Eco2.User user)
@@
   )
   (setup
-    (last_trace_width 1)
+    (last_trace_width 0.25)
     (user_trace_width 0.25)
     (user_trace_width 0.5)
@@
     (at 85 90 90)
     (descr "WireConnection with 2mm drill")
-    (fp_text reference CAPS (at 5 -3 90) (layer F.SilkS)
+    (fp_text reference P4 (at 5 -3 90) (layer F.SilkS)
       (effects (font (size 1 1) (thickness 0.15)))
     )
@@
     (at 125 44)
     (descr "WireConnection with 2mm drill")
-    (fp_text reference SOL (at 5 -2) (layer F.SilkS)
+    (fp_text reference P1 (at 5 -2) (layer F.SilkS)
       (effects (font (size 1 1) (thickness 0.15)))
     )
@@
     (at 85 70 90)
     (descr "WireConnection with 2mm drill")
-    (fp_text reference POLOLU (at 5 -3 90) (layer F.SilkS)
+    (fp_text reference P2 (at 5 -3 90) (layer F.SilkS)
       (effects (font (size 1 1) (thickness 0.15)))
     )
@@
     (at 105 44)
     (descr "WireConnection with 2mm drill")
-    (fp_text reference BATT (at 5 -2) (layer F.SilkS)
+    (fp_text reference P3 (at 5 -2) (layer F.SilkS)
       (effects (font (size 1 1) (thickness 0.15)))
     )
@@
     (at 86 44)
     (descr "WireConnection with 2mm drill")
-    (fp_text reference MEGA (at 5 -2) (layer F.SilkS)
+    (fp_text reference P5 (at 5 -2) (layer F.SilkS)
       (effects (font (size 1 1) (thickness 0.15)))
     )
@@
   (module Wire_Pads:SolderWirePad_single_1-2mmDrill (layer F.Cu)
     (at 84 51)
-    (fp_text reference FBK (at -3 0 90) (layer F.SilkS)
-      (effects (font (size 1 1) (thickness 0.15)))
-    )
+    (fp_text reference P6 (at -3 0 90) (layer F.SilkS)
+      (effects (font (size 1 1) (thickness 0.15)))
+    )

Commit message: correct new PSB with net-tie on master
Parts:
- added W1: NET-TIE, conn-test:NET-TIE-1mm, F.Cu at (91.0, 96.0)
Connections:
- C1 pad 2: GND -> /Ref_gnd
- C2 pad 2: GND -> /Ref_gnd
- IC1 pad 22: GND -> /Ref_gnd
- IC1 pad 8: GND -> /Ref_gnd
Routing:
- net /Ref_gnd: track 0.00 -> 57.4 mm
- net GND: track 10.5 -> 10.1 mm, vias 0 -> 1
Changed lines of the file:
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@@
 (kicad_pcb (version 4) (host pcbnew 4.0.2+dfsg1-stable)
   (general
-    (links 38)
+    (links 39)
     (no_connects 0)
-    (area 76 37 147.000001 123.000001)
+    (area 79.949999 39.949999 140.050001 120.050001)
     (thickness 1.6)
     (drawings 15)
-    (tracks 104)
+    (tracks 122)
     (zones 0)
-    (modules 20)
-    (nets 30)
+    (modules 21)
+    (nets 31)
   )
   (page A4)
@@
   )
   (layers
-    (0 F.Cu signal)
-    (31 B.Cu signal)
-    (32 B.Adhes user)
-    (33 F.Adhes user)
-    (34 B.Paste user)
-    (35 F.Paste user)
+    (0 F.Cu signal hide)
+    (31 B.Cu signal hide)
+    (32 B.Adhes user hide)
+    (33 F.Adhes user hide)
+    (34 B.Paste user hide)
+    (35 F.Paste user hide)
     (36 B.SilkS user)
     (37 F.SilkS user)
-    (38 B.Mask user)
-    (39 F.Mask user)
-    (40 Dwgs.User user)
+    (38 B.Mask user hide)
+    (39 F.Mask user hide)
+    (40 Dwgs.User user hide)
     (41 Cmts.User user hide)
-    (42 Eco1.User user)
-    (43 Eco2.User user)
+    (42 Eco1.User user hide)
+    (43 Eco2.User user hide)
     (44 Edge.Cuts user)
-    (45 Margin user)
-    (46 B.CrtYd user)
-    (47 F.CrtYd user)
+    (45 Margin user hide)
+    (46 B.CrtYd user hide)
+    (47 F.CrtYd user hide)
     (48 B.Fab user hide)
     (49 F.Fab user hide)
   )
   (setup
-    (last_trace_width 0.25)
+    (last_trace_width 0.75)
     (user_trace_width 0.25)
     (user_trace_width 0.5)
@@
   (net 28 /MSFT_SOLAR_S)
   (net 29 /MEGA-)
+  (net 30 /Ref_gnd)
   (net_class Default "This is the default net class."
     (clearance 0.3)
@@
     (add_net /D5)
     (add_net /MEGA_FBK)
+    (add_net /Ref_gnd)
     (add_net "Net-(C1-Pad1)")
     (add_net "Net-(C2-Pad1)")
@@
       (net 1 "Net-(C1-Pad1)"))
     (pad 2 thru_hole circle (at 2.5 0) (size 1.3 1.3) (drill 0.8001) (layers *.Cu *.Mask F.SilkS)
-      (net 2 GND))
+      (net 30 /Ref_gnd))
     (model Capacitors_ThroughHole.3dshapes/C_Disc_D3_P2.5.wrl
       (at (xyz 0.0492126 0 0))
@@
       (net 3 "Net-(C2-Pad1)"))
     (pad 2 thru_hole circle (at 2.5 0 180) (size 1.3 1.3) (drill 0.8001) (layers *.Cu *.Mask F.SilkS)
-      (net 2 GND))
+      (net 30 /Ref_gnd))
     (model Capacitors_ThroughHole.3dshapes/C_Disc_D3_P2.5.wrl
       (at (xyz 0.049213 0 0))
@@
       (net 11 +5V))
     (pad 8 thru_hole oval (at 0 17.78) (size 2.3 1.6) (drill 0.8) (layers *.Cu *.Mask F.SilkS)
-      (net 2 GND))
+      (net 30 /Ref_gnd))
     (pad 9 thru_hole oval (at 0 20.32) (size 2.3 1.6) (drill 0.8) (layers *.Cu *.Mask F.SilkS)
       (net 3 "Net-(C2-Pad1)"))
@@
       (net 21 "Net-(IC1-Pad21)"))
     (pad 22 thru_hole oval (at 7.62 15.24) (size 2.3 1.6) (drill 0.8) (layers *.Cu *.Mask F.SilkS)
-      (net 2 GND))
+      (net 30 /Ref_gnd))
     (pad 23 thru_hole oval (at 7.62 12.7) (size 2.3 1.6) (drill 0.8) (layers *.Cu *.Mask F.SilkS)
       (net 22 /A0))
@@
       (net 1 "Net-(C1-Pad1)"))
   )
+  (module conn-test:NET-TIE-1mm (layer F.Cu)
+    (at 91 96)
+    (fp_text reference W1 (at 0 -2) (layer F.SilkS) hide
+      (effects (font (size 0.8 0.8) (thickness 0.15)))
+    )
+    (fp_text value NET-TIE (at 0 2) (layer F.Fab) hide
+      (effects (font (size 0.8 0.8) (thickness 0.15)))
+    )
+    (fp_line (start -0.95 0) (end 0.95 0) (layer F.Cu) (width 1))
+    (pad 1 smd circle (at -0.95 0) (size 1 1) (layers F.Cu)
+      (net 2 GND))
+    (pad 2 smd circle (at 0.95 0) (size 1 1) (layers F.Cu)
+      (net 30 /Ref_gnd))
+  )
   (gr_text + (at 87 87) (layer F.SilkS)
     (effects (font (size 1.5 1.5) (thickness 0.3)))
@@
   (segment (start 103.35 100.86) (end 105 100.86) (width 0.5) (layer F.Cu) (net 1))
   (segment (start 97 107.44094) (end 102.5 101.94094) (width 0.5) (layer F.Cu) (net 1))
-  (segment (start 104.65 95.78) (end 105 95.78) (width 0.5) (layer F.Cu) (net 2))
+  (via (at 90.05 96) (size 0.9) (drill 0.6) (layers F.Cu B.Cu) (net 2))
   (segment (start 115.16 44) (end 112.46 46.7) (width 1.5) (layer F.Cu) (net 2))
   (segment (start 112.46 46.7) (end 112.46 53) (width 1.5) (layer F.Cu) (net 2))
@@
   (segment (start 96.16 44) (end 96.16 52.7) (width 1.5) (layer F.Cu) (net 29))
   (segment (start 96.16 52.7) (end 96.46 53) (width 1.5) (layer F.Cu) (net 29))
+  (segment (start 112.62 93.24) (end 112.5 93) (width 0.75) (layer B.Cu) (net 30) (status 80000))
+  (segment (start 112.5 93) (end 109.5 96) (width 0.75) (layer B.Cu) (net 30) (status 80000))
+  (segment (start 109.5 96) (end 105 96) (width 0.75) (layer B.Cu) (net 30) (status 80000))
+  (segment (start 105 96) (end 105 95.78) (width 0.75) (layer B.Cu) (net 30) (status 80000))
+  (segment (start 105 95.78) (end 105 96) (width 0.75) (layer B.Cu) (net 30) (status 80000))
+  (segment (start 105 96) (end 103.5 94.5) (width 0.75) (layer B.Cu) (net 30) (status 80000))
+  (segment (start 103.5 94.5) (end 96 94.5) (width 0.75) (layer B.Cu) (net 30) (status 80000))
+  (segment (start 96 94.5) (end 96 95) (width 0.75) (layer B.Cu) (net 30) (status 80000))
+  (segment (start 96 95) (end 95 96) (width 0.75) (layer B.Cu) (net 30) (status 80000))
+  (segment (start 95 96) (end 95 96.5) (width 0.75) (layer F.Cu) (net 30))
+  (segment (start 95 96.5) (end 92.5 99) (width 0.75) (layer F.Cu) (net 30))
+  (segment (start 98.5 118.5) (end 98.5 115) (width 0.75) (layer F.Cu) (net 30))
+  (segment (start 99 119) (end 98.5 118.5) (width 0.75) (layer F.Cu) (net 30))
+  (segment (start 95.5 119) (end 99 119) (width 0.75) (layer F.Cu) (net 30))
+  (segment (start 92.5 116) (end 95.5 119) (width 0.75) (layer F.Cu) (net 30))
+  (segment (start 92.5 99) (end 92.5 116) (width 0.75) (layer F.Cu) (net 30))
+  (segment (start 95 96) (end 91.95 96) (width 0.75) (layer F.Cu) (net 30))
+  (segment (start 104.65 95.78) (end 105 95.78) (width 0.5) (layer F.Cu) (net 30))
   (zone (net 2) (net_name GND) (layer B.Cu) (hatch edge 0.508)
     (connect_pads (clearance 0.508))

Commit message: files to send to Olav for double checking
Parts:
- U1: value IRLB-8721_SOL -> IRLB_8721_SOL
- U2: value IRLB-8721_MEGA -> IRLS-8721_MEGA
- moved R6 10.0 mm to (94.0, 60.0), turned to 0 degrees
- moved U1 8.00 mm to (123.0, 53.0), turned to 0 degrees
- moved U2 0.71 mm to (99.5, 52.5), turned to 0 degrees
Connections:
- U1 pad 2: /MSFT_SOLAR_S -> GND
- U1 pad 3: GND -> /MSFT_SOLAR_S
- U2 pad 2: GND -> /MEGA-
- U2 pad 3: /MEGA- -> GND
Routing:
- net /D5: track 129.2 -> 106.7 mm
- net GND: track 10.1 -> 0.00 mm
- net /MSFT_SOLAR_S: track 58.1 -> 61.4 mm
- net Net-(C1-Pad1): track 18.8 -> 21.6 mm
- net /Ref_gnd: track 57.4 -> 59.9 mm, vias 0 -> 1
- net +5V: track 136.1 -> 137.4 mm
- net /D3: track 71.1 -> 70.0 mm
- net /MEGA-: track 9.12 -> 9.98 mm
- net /A0: track 72.9 -> 73.7 mm
- added copper zone on F.Cu, net +5V
Other:
- board size 60 x 80 mm -> 60 x 81.5 mm
- board text added: "Power manager v1.1 Jean Rabault, UiO 12-2017"
