File: PCB_electronics/power_controller_v3/power_controller_SMD.kicad_pcb (KiCad board)
At the start: 2 copper layers, 49 x 66 mm, 21 parts, among them J1 DIP-BLACK-MALE-HEADER_2X3P-2.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, J2 SCREW-TERMINAL-GREEN_2P-5.0_, J3 SCREW-TERMINAL-GREEN_2P-5.0_, J4 SCREW-TERMINAL-GREEN_2P-5.0_, J5 SCREW-TERMINAL-GREEN_2P-5.0_, J6 SCREW-TERMINAL-GREEN_3P-5.0_, P1 CONN_01X06, P2 CONN_01X02, P3 CONN_01X06, Q1 SMD-MOSFET-N-CH-20V-2.1A-CJ23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

Commit message: ready to generate first gerbers for test for power manager v3
Other:
- board text added: "+"
- board text added: "-"
- board text added: "BATT"
- board text added: "CAPS"
- board text added: "FBK"
- board text added: "ICSP"
- board text added: "MEGA"
- board text added: "MISO"
- board text added: "MOSI"
- board text added: "POLOLU"
- board text added: "Power Manager v3.1 Jean Rabault, UiO 12-2017"
- board text added: "RST"
- board text added: "SCK"
- board text added: "SOL"
