File: PCB_electronics/Logger_and_power_v1/Power_part.sch (KiCad schematic (older format))
At the start: 19 parts, among them IC1 ATMEGA328-P, P1 SOLAR_PANEL, P2 5V_pololu, P3 BATT, P4 SUPERCAPS, U1 IRLB_8721_SOL, U2 IRLS-8721_MEGA, Y1 16MHz

Commit message: ready to try to shift the power controller
Parts:
- W1: footprint conn-test:NET-TIE -> Oddities:NetTie-I_Connected
Changed lines of the file:
@@
 F 0 "W1" H 1600 5350 50  0000 C CNN
 F 1 "NET-TIE" H 1600 5250 50  0000 C CNN
-F 2 "conn-test:NET-TIE" H 1600 5000 50  0001 C CNN
+F 2 "Oddities:NetTie-I_Connected" H 1600 5000 50  0001 C CNN
 F 3 "" H 1600 5100 60  0000 C CNN
 	1    1600 5100

Commit message: now pololu on PCB; need to export gerbers still
Parts:
- added P19: header_pololu_in, symbol CONN_01X05
- added P20: header_pololu_out, symbol CONN_01X04
Connections:
- net +5V: now also P20.1 (P1), P20.2 (P2)
- net Batt_plus: now also P19.4 (P4), P19.5 (P5)
- net GND: now also P19.2 (P2), P19.3 (P3), P20.3 (P3), P20.4 (P4)
- new net enable_default_on: P19.1 (P1)
- no-connect marks 15 -> 17
Changed lines of the file:
@@
 	-1   0    0    1
 $EndComp
+NoConn ~ 10200 3750
+$Comp
+L CONN_01X05 P19
+U 1 1 5D40578E
+P 8150 950
+F 0 "P19" H 8150 1250 50  0000 C CNN
+F 1 "header_pololu_in" V 8250 950 50  0000 C CNN
+F 2 "" H 8150 950 50  0000 C CNN
+F 3 "" H 8150 950 50  0000 C CNN
+	1    8150 950
+	1    0    0    -1
+$EndComp
+$Comp
+L CONN_01X04 P20
+U 1 1 5D405903
+P 8750 900
+F 0 "P20" H 8750 1150 50  0000 C CNN
+F 1 "header_pololu_out" V 8850 900 50  0000 C CNN
+F 2 "" H 8750 900 50  0000 C CNN
+F 3 "" H 8750 900 50  0000 C CNN
+	1    8750 900
+	-1   0    0    1
+$EndComp
+Wire Wire Line
+	8950 950  9200 950
+Wire Wire Line
+	9200 950  9200 1050
+Wire Wire Line
+	9200 1050 8950 1050
+Wire Wire Line
+	9200 850  8950 850
+Wire Wire Line
+	9200 750  9200 850
+Wire Wire Line
+	9200 750  8950 750
+Connection ~ 9200 800
+Wire Wire Line
+	9200 1000 9900 1000
+Connection ~ 9200 1000
+$Comp
+L GND #PWR019
+U 1 1 5D405E2B
+P 9600 700
+F 0 "#PWR019" H 9600 450 50  0001 C CNN
+F 1 "GND" H 9600 550 50  0000 C CNN
+F 2 "" H 9600 700 50  0000 C CNN
+F 3 "" H 9600 700 50  0000 C CNN
+	1    9600 700
+	1    0    0    -1
+$EndComp
+Wire Wire Line
+	9200 800  9350 800
+Wire Wire Line
+	9350 800  9350 700
+Wire Wire Line
+	9350 700  9600 700
+$Comp
+L +5V #PWR020
+U 1 1 5D406012
+P 9900 1000
+F 0 "#PWR020" H 9900 850 50  0001 C CNN
+F 1 "+5V" H 9900 1140 50  0000 C CNN
+F 2 "" H 9900 1000 50  0000 C CNN
+F 3 "" H 9900 1000 50  0000 C CNN
+	1    9900 1000
+	1    0    0    -1
+$EndComp
+NoConn ~ 7950 750
+Text Label 7950 750  2    60   ~ 0
+enable_default_on
+Wire Wire Line
+	7550 850  7950 850
+Wire Wire Line
+	7750 850  7750 950
+Wire Wire Line
+	7750 950  7950 950
+Wire Wire Line
+	7950 1050 7750 1050
+Wire Wire Line
+	7750 1050 7750 1150
+Wire Wire Line
+	7350 1150 7950 1150
+Connection ~ 7750 850
+$Comp
+L GND #PWR021
+U 1 1 5D406578
+P 7550 850
+F 0 "#PWR021" H 7550 600 50  0001 C CNN
+F 1 "GND" H 7550 700 50  0000 C CNN
+F 2 "" H 7550 850 50  0000 C CNN
+F 3 "" H 7550 850 50  0000 C CNN
+	1    7550 850
+	1    0    0    -1
+$EndComp
+Connection ~ 7750 1150
+Text Label 7350 1150 2    60   ~ 0
+COMMON_BAT+_SOL+
 $EndSCHEMATC

Commit message: PCB with pololu support, for order 07-2019
Parts:
- P19: footprint (none) -> Pin_Headers:Pin_Header_Straight_1x05
- P20: footprint (none) -> Pin_Headers:Pin_Header_Straight_1x04
Changed lines of the file:
@@
 F 0 "P19" H 8150 1250 50  0000 C CNN
 F 1 "header_pololu_in" V 8250 950 50  0000 C CNN
-F 2 "" H 8150 950 50  0000 C CNN
+F 2 "Pin_Headers:Pin_Header_Straight_1x05" H 8150 950 50  0001 C CNN
 F 3 "" H 8150 950 50  0000 C CNN
 	1    8150 950
@@
 F 0 "P20" H 8750 1150 50  0000 C CNN
 F 1 "header_pololu_out" V 8850 900 50  0000 C CNN
-F 2 "" H 8750 900 50  0000 C CNN
+F 2 "Pin_Headers:Pin_Header_Straight_1x04" H 8750 900 50  0001 C CNN
 F 3 "" H 8750 900 50  0000 C CNN
 	1    8750 900

Commit message: working on the pcb v3.5
Parts:
- R1: value 5.6k -> 56k
- R2: value 3.9k -> 39k
- R3, R5, R6, R7: value 50k -> 47k
Changed lines of the file:
@@
 P 4350 3150
 F 0 "R3" V 4430 3150 50  0000 C CNN
-F 1 "50k" V 4350 3150 50  0000 C CNN
+F 1 "47k" V 4350 3150 50  0000 C CNN
 F 2 "Resistors_ThroughHole:Resistor_Horizontal_RM10mm" V 4280 3150 50  0001 C CNN
 F 3 "" H 4350 3150 50  0000 C CNN
@@
 P 5500 4500
 F 0 "R5" V 5580 4500 50  0000 C CNN
-F 1 "50k" V 5500 4500 50  0000 C CNN
+F 1 "47k" V 5500 4500 50  0000 C CNN
 F 2 "Resistors_ThroughHole:Resistor_Horizontal_RM10mm" V 5430 4500 50  0001 C CNN
 F 3 "" H 5500 4500 50  0000 C CNN
@@
 P 5550 5650
 F 0 "R6" V 5630 5650 50  0000 C CNN
-F 1 "50k" V 5550 5650 50  0000 C CNN
+F 1 "47k" V 5550 5650 50  0000 C CNN
 F 2 "Resistors_ThroughHole:Resistor_Horizontal_RM10mm" V 5480 5650 50  0001 C CNN
 F 3 "" H 5550 5650 50  0000 C CNN
@@
 P 7850 5650
 F 0 "R7" V 7930 5650 50  0000 C CNN
-F 1 "50k" V 7850 5650 50  0000 C CNN
+F 1 "47k" V 7850 5650 50  0000 C CNN
 F 2 "Resistors_ThroughHole:Resistor_Horizontal_RM10mm" V 7780 5650 50  0001 C CNN
 F 3 "" H 7850 5650 50  0000 C CNN
@@
 P 3700 5550
 F 0 "R2" V 3780 5550 50  0000 C CNN
-F 1 "3.9k" V 3700 5550 50  0000 C CNN
+F 1 "39k" V 3700 5550 50  0000 C CNN
 F 2 "Resistors_ThroughHole:Resistor_Horizontal_RM10mm" V 3630 5550 50  0001 C CNN
 F 3 "" H 3700 5550 50  0000 C CNN
@@
 P 3700 5050
 F 0 "R1" V 3780 5050 50  0000 C CNN
-F 1 "5.6k" V 3700 5050 50  0000 C CNN
+F 1 "56k" V 3700 5050 50  0000 C CNN
 F 2 "Resistors_ThroughHole:Resistor_Horizontal_RM10mm" V 3630 5050 50  0001 C CNN
 F 3 "" H 3700 5050 50  0000 C CNN
